File: Diagrams/KiCAD/V3-working/V3.sch (KiCad schematic (older format))
At the start: 41 parts, among them U2 NodeMCU_1.0_(ESP-12E), U3 74HC595, U4 74HC595

Commit message: Updated diagrams
Parts:
- gave numbers to parts that had none: 34
Connections:
- net labels added: GY, OUT, VI
